File: Schaltung/att/att.kicad_sch (KiCad schematic)
At the start: 9 parts, among them J1 Screw_Terminal_01x02, J2 Dsiplay, J3 Drehgeber, J4 Controller, J5 R&S Attenuator 26.5 GHz

Commit message: kicad
Parts:
- J1: value Screw_Terminal_01x02 -> 12V Power supply
- J3: value Drehgeber -> dB Drehgeber
- J4: value Controller -> ESP-Controller
Connections:
- net GND: now also J5.4 (Pin_4), J5.7 (Pin_7); no longer J5.2 (Pin_2), J5.9 (Pin_9)
- net at J5.10 (Pin_10): now also U3. (GND)
- net at J5.5 (Pin_5): now also U3. (GND)
- new net: J1.1 (Pin_1), U1. (GND), U2. (GND)
- new net: J5.2 (Pin_2), U3. (GND)
- new net: J5.9 (Pin_9), U3. (GND)
Other:
- note added: "0.5"
- note added: "10dB"
- note added: "2026/04"
- note added: "20dB"
- note added: "40dB"
- note added: "5V"
- note added: "Attenuator Controller"
- note added: "OE5RNL & OE5NVL"
- note added: "Vs"
- moved on the sheet: A1, J1, J2, J3, J4, J5, U1, U2, U3
