File: Schaltung/att_135/att.kicad_pcb (KiCad board)
At the start: 2 copper layers, 99 x 92 mm, 8 parts, among them U10 DRV8871DDA, U4 DRV8871DDA, U5 DRV8871DDA, U6 DRV8871DDA, U7 DRV8871DDA, U8 DRV8871DDA, U9 DRV8871DDA

Commit message: 1
Parts:
- removed U10, U8, U9: DRV8871DDA, Package_SO:Texas_HTSOP-8-1EP_3.9x4.9mm_P1.27mm_EP2.95x4.9mm_Mask2.4x3.1mm_ThermalVias
- added C1: 100nF, Resistor_SMD:R_0805_2012Metric, F.Cu at (105.6, 71.9)
- added J1: 12V Power supply, TerminalBlock_MetzConnect:TerminalBlock_MetzConnect_Type055_RT01502HDWU_1x02_P5.00mm_Horizontal, F.Cu at (51.9, 64.5)
- added R1: 15k, Resistor_SMD:R_0805_2012Metric, F.Cu at (105.7, 74.6)
- added U1: DRV8871DDA, Package_SO:Texas_HTSOP-8-1EP_3.9x4.9mm_P1.27mm_EP2.95x4.9mm_Mask2.4x3.1mm_ThermalVias, F.Cu at (105.6, 62.8)
- added U2: DRV8871DDA, Package_SO:Texas_HTSOP-8-1EP_3.9x4.9mm_P1.27mm_EP2.95x4.9mm_Mask2.4x3.1mm_ThermalVias, F.Cu at (124.6, 87.2)
- added U20: ~, RNL_ATT:MP1584EN_module, F.Cu at (74.7, 65.0)
- added U3: DRV8871DDA, Package_SO:Texas_HTSOP-8-1EP_3.9x4.9mm_P1.27mm_EP2.95x4.9mm_Mask2.4x3.1mm_ThermalVias, F.Cu at (118.0, 87.2)
- added U30: ~, RNL_ATT:ttl_converter, F.Cu at (92.0, 31.2)
- moved U6 51.2 mm to (98.1, 87.2), turned to -90 degrees
- moved U4 46.5 mm to (111.3, 87.2), turned to -90 degrees
- moved U5 40.5 mm to (104.7, 87.2), turned to -90 degrees
- moved A1 38.3 mm to (155.8, 72.5), turned to -90 degrees
- moved U7 27.5 mm to (91.4, 87.2), turned to -90 degrees
Connections:
- U4 pad 2: Net-(A1-GPIO28_ADC2) -> Net-(A1-GPIO9)
- U4 pad 3: Net-(A1-GPIO27_ADC1) -> Net-(A1-GPIO8)
- U4 pad 4: unconnected-(U4-ILIM-Pad4) -> Net-(U4-ILIM)
- U5 pad 2: Net-(A1-GPIO26_ADC0) -> Net-(A1-GPIO28_ADC2)
- U5 pad 3: Net-(A1-GPIO22) -> Net-(A1-GPIO27_ADC1)
- U5 pad 4: unconnected-(U5-ILIM-Pad4) -> Net-(U5-ILIM)
- U6 pad 2: Net-(A1-GPIO17) -> Net-(A1-GPIO26_ADC0)
- U6 pad 3: Net-(A1-GPIO16) -> Net-(A1-GPIO22)
- U6 pad 4: unconnected-(U6-ILIM-Pad4) -> Net-(U6-ILIM)
- U7 pad 2: Net-(A1-GPIO15) -> Net-(A1-GPIO17)
- U7 pad 3: Net-(A1-GPIO14) -> Net-(A1-GPIO16)
- U7 pad 4: unconnected-(U7-ILIM-Pad4) -> Net-(U7-ILIM)
Routing:
- net Net-(A1-GPIO11): track 13.9 -> 57.6 mm
- net Net-(A1-GPIO10): track 14.4 -> 58.1 mm
- net Net-(A1-GPIO12): track 29.5 -> 0.00 mm
- net Net-(A1-GPIO13): track 29.3 -> 0.00 mm
- net Net-(A1-GPIO28_ADC2): track 26.1 -> 0.00 mm
- net Net-(A1-GPIO27_ADC1): track 25.1 -> 0.00 mm
- net Net-(A1-GPIO14): track 20.1 -> 0.00 mm
- net Net-(A1-GPIO15): track 19.6 -> 0.00 mm
- net Net-(A1-GPIO26_ADC0): track 13.4 -> 0.00 mm
- net Net-(A1-GPIO22): track 13.0 -> 0.00 mm
- net Net-(A1-GPIO9): track 11.1 -> 0.00 mm
- net Net-(A1-GPIO8): track 10.3 -> 0.00 mm
- net GND: track 0.00 -> 9.60 mm
- net Net-(U1-ILIM): track 0.00 -> 9.59 mm, vias 0 -> 2
Other:
- board size 99 x 92 mm -> 136 x 39 mm
