File: Schaltung/att_135/att.kicad_sch (KiCad schematic)
At the start: 24 parts, among them J1 12V Power supply, J10 RF_ON_OFF, J11 40dB_B, J12 10dB, J13 ATT_SEL, J2 Dsiplay, J3 dB Drehgeber, J4 ESP-Controller, J5 R&S Attenuator 26.5 GHz, J6 20dB_A, J7 40dB_A, J8 20dB_B, J9 5dB, U10 DRV8871DDA, U4 DRV8871DDA, U5 DRV8871DDA, U6 DRV8871DDA, U7 DRV8871DDA, U8 DRV8871DDA, U9 DRV8871DDA

Commit message: 1
Parts:
- added C1: 100nF, Resistor_SMD:R_0805_2012Metric, symbol Device:C
- added C10, C20_1: 47uF 50V, symbol Device:C_Polarized
- added C2, C5, C6: 100 nF, symbol Device:C
- added C3, C4, C7: 100nF, symbol Device:C
- added J14: Conn_01x02_Pin, symbol Connector:Conn_01x02_Pin
- added R1, R2, R3, R5, R6, R7: 15k, symbol Device:R
- added R4: 15K, symbol Device:R
- J1: footprint (none) -> TerminalBlock_MetzConnect:TerminalBlock_MetzConnect_Type055_RT01502HDWU_1x02_P5.00mm_Horizontal
- U20: renamed from U2; footprint (none) -> RNL_ATT:MP1584EN_module
- U30: renamed from U3; footprint (none) -> RNL_ATT:ttl_converter
- renumbered U8 to U1, U1 to U10, U10 to U2, U7 to U3, U9 to U4, U4 to U5, U5 to U6, U6 to U7
Connections:
- net +15V: now also C10.1, C20_1.1
- net GND: now also C1.1, C10.2, C2.1, C20_1.2, C3.2, C4.2, C5.2, C6.2, C7.2, J14.1 (Pin_1), J14.2 (Pin_2), R1.2, R2.1, R3.2, R4.2, R5.2, R6.2, R7.2
- net at U7.4 (ILIM): now also C7.1, R7.1
- net at U2.4 (ILIM): now also C2.2, R2.2
- net at U5.4 (ILIM): now also C5.1, R5.1
- net at U4.4 (ILIM): now also C4.1, R4.1
- net at U3.4 (ILIM): now also C3.1, R3.1
- net at U6.4 (ILIM): now also C6.1, R6.1
- net at U1.4 (ILIM): now also C1.2, R1.1
- new net: J1.1 (Pin_1), U10. (GND), U20. (GND)
Other:
- moved on the sheet: A1, J1, J10, J11, J12, J13, J2, J3, J4, J5, J6, J7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
