File: Schaltung/att.kicad_pcb (KiCad board)
At the start: 2 copper layers, 95.2 x 75 mm, 51 parts, among them J1 12V Power supply, J10 RF_ON_OFF, J11 40dB_B, J12 10dB, J15 5V für ESP Panel, J16 Conn_02x05_Odd_Even, J17 20dB_A, J18 20dB_A, J2 Dsiplay, J3 dB Drehgeber, J4 ESP-Controller, J6 20dB_A, J7 40dB_A, J8 20dB_B, J9 5dB, U1 DRV8871DDA, U12 DRV8871DDA, U2 DRV8871DDA, U3 DRV8871DDA, U4 DRV8871DDA, U5 DRV8871DDA, U6 DRV8871DDA, U7 DRV8871DDA, U9 DRV8871DDA

Commit message: pcb
Parts:
- moved J12 93.7 mm to (55.7, 117.7), turned to 180 degrees
- moved J11 93.4 mm to (55.5, 111.1), turned to 180 degrees
- moved J10 92.8 mm to (56.0, 103.2), turned to 180 degrees
- moved J1 68.3 mm to (103.9, 52.7), turned to 0 degrees
- moved U5 57.2 mm to (64.6, 102.5), turned to 180 degrees
- moved C11 56.4 mm to (164.5, 78.1), turned to 180 degrees
- moved U6 55.7 mm to (64.7, 109.9), turned to 180 degrees
- moved C5 51.0 mm to (70.7, 101.4), turned to 90 degrees
- moved C6 49.1 mm to (71.0, 108.9), turned to 90 degrees
- moved U7 48.8 mm to (64.9, 117.4), turned to 180 degrees
- moved R5 45.5 mm to (73.1, 101.4), turned to 90 degrees
- moved C12 43.5 mm to (159.9, 122.5)
- moved R6 43.0 mm to (73.8, 108.8), turned to 90 degrees
- moved J2 42.2 mm to (103.1, 70.3)
- moved C7 41.5 mm to (74.5, 115.7), turned to 90 degrees
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Routing:
- net GND: track 54.5 -> 208.0 mm, vias 7 -> 8
- net +15V-24V: track 112.4 -> 0.00 mm, vias 1 -> 0
- net +3.3V: track 91.6 -> 45.4 mm
- net +5V: track 77.8 -> 37.8 mm, vias 1 -> 0
- net /10dB: track 28.6 -> 0.00 mm
- net /40dBb: track 21.8 -> 0.00 mm
- net Net-(A1-GPIO1): track 21.8 -> 0.00 mm
- net Net-(A1-GPIO13): track 19.1 -> 0.00 mm, vias 1 -> 0
- net /40dBa: track 17.4 -> 0.00 mm
- net Net-(A1-GPIO6): track 0.28 -> 11.5 mm, vias 0 -> 1
- net Net-(A1-GPIO7): track 0.42 -> 9.08 mm, vias 0 -> 1
- net Net-(J18-Pin_2): track 8.47 -> 0.00 mm
- net Net-(J18-Pin_1): track 8.47 -> 0.00 mm
- net +15V: track 124.3 -> 116.2 mm, vias 3 -> 1
- net Net-(U4-ILIM): track 6.47 -> 0.00 mm
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Other:
- board size 95.2 x 75 mm -> 84.7 x 75 mm

Commit message: schaltung PCB
Parts:
- removed J10: RF_ON_OFF, Connector_PinHeader_2.54mm:PinHeader_1x02_P2.54mm_Vertical
- removed J11: 40dB_B, Connector_PinHeader_2.54mm:PinHeader_1x02_P2.54mm_Vertical
- removed J12: 10dB, Connector_PinHeader_2.54mm:PinHeader_1x02_P2.54mm_Vertical
- removed J15: 5V für ESP Panel, Connector_PinHeader_2.54mm:PinHeader_1x02_P2.54mm_Vertical
- removed J17, J18, J6: 20dB_A, Connector_PinHeader_2.54mm:PinHeader_1x02_P2.54mm_Vertical
- removed J7: 40dB_A, Connector_PinHeader_2.54mm:PinHeader_1x02_P2.54mm_Vertical
- removed J8: 20dB_B, Connector_PinHeader_2.54mm:PinHeader_1x02_P2.54mm_Vertical
- removed J9: 5dB, Connector_PinHeader_2.54mm:PinHeader_1x02_P2.54mm_Vertical
- added U13: ~, 0_RNL_ATT:SIL_18, F.Cu at (56.6, 73.1)
- C4: footprint Capacitor_SMD:C_0805_2012Metric_Pad1.18x1.45mm_HandSolder -> Resistor_SMD:R_0805_2012Metric
- J4: footprint Connector_PinHeader_2.54mm:PinHeader_1x03_P2.54mm_Vertical -> Connector_PinHeader_2.54mm:PinHeader_1x04_P2.54mm_Vertical
- R1, R4, R8, R9: footprint Resistor_SMD:R_0805_2012Metric_Pad1.20x1.40mm_HandSolder -> Resistor_SMD:R_0805_2012Metric
- U12: value DRV8871DDA -> ~; footprint Package_SO:Texas_HTSOP-8-1EP_3.9x4.9mm_P1.27mm_EP2.95x4.9mm_Mask2.4x3.1mm_ThermalVias -> 0_RNL_ATT:DC-DC_12_24
- U8: value ~ -> DRV8871DDA; footprint 0_RNL_ATT:DC-DC_12_24 -> Package_SO:Texas_HTSOP-8-1EP_3.9x4.9mm_P1.27mm_EP2.95x4.9mm_Mask2.4x3.1mm_ThermalVias
- moved C21 169.1 mm to (104.9, 54.1)
- moved C12 83.7 mm to (77.1, 109.7), turned to 90 degrees
- moved C11 77.9 mm to (96.2, 40.7), turned to -90 degrees
- moved U8 70.7 mm to (65.0, 107.6), turned to 180 degrees
- moved U12 67.6 mm to (101.0, 114.4), turned to 90 degrees
- moved U9 49.5 mm to (65.0, 114.7)
- moved U10 42.1 mm to (111.5, 71.1), turned to 0 degrees
- moved J3 27.9 mm to (128.6, 85.1)
- moved J2 25.5 mm to (128.6, 68.8), turned to 180 degrees
- moved U3 22.7 mm to (65.3, 72.6)
- moved U2 22.2 mm to (65.4, 65.5)
- moved U1 21.7 mm to (65.5, 58.5)
- moved C20 21.7 mm to (108.1, 40.9), turned to -90 degrees
- moved U11 19.6 mm to (113.5, 88.8), turned to 0 degrees
- moved R7 18.1 mm to (71.1, 97.8)
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Connections:
- A1 pad 1: Net-(A1-GPIO0) -> /TX
- A1 pad 2: Net-(A1-GPIO1) -> /RX
- C1 pad 2: Net-(U1-ILIM) -> Net-(U4-ILIM)
- C2 pad 2: Net-(U2-ILIM) -> Net-(U5-ILIM)
- C20 pad 1: +15V-24V -> unconnected-(C20-Pad1)
- C20 pad 2: GND -> unconnected-(C20-Pad2)
- C3 pad 1: Net-(U3-ILIM) -> Net-(U6-ILIM)
- C4 pad 1: Net-(U4-ILIM) -> Net-(U3-ILIM)
- C5 pad 1: Net-(U5-ILIM) -> Net-(U9-ILIM)
- C6 pad 1: Net-(U6-ILIM) -> Net-(U8-ILIM)
- C8 pad 2: Net-(U9-ILIM) -> Net-(U2-ILIM)
- C9 pad 2: Net-(U12-ILIM) -> Net-(U1-ILIM)
- J4 pad 1: Net-(A1-GPIO0) -> +5V
- J4 pad 2: Net-(A1-GPIO1) -> /TX
- J4 pad 3: GND -> /RX
- R1 pad 1: Net-(U1-ILIM) -> Net-(U4-ILIM)
- R2 pad 2: Net-(U2-ILIM) -> Net-(U5-ILIM)
- R3 pad 1: Net-(U3-ILIM) -> Net-(U6-ILIM)
- R4 pad 1: Net-(U4-ILIM) -> Net-(U3-ILIM)
- R5 pad 1: Net-(U5-ILIM) -> Net-(U9-ILIM)
- R6 pad 1: Net-(U6-ILIM) -> Net-(U8-ILIM)
- R8 pad 1: Net-(U9-ILIM) -> Net-(U2-ILIM)
- R9 pad 1: Net-(U12-ILIM) -> Net-(U1-ILIM)
- U1 pad 2: Net-(A1-GPIO11) -> Net-(A1-GPIO3)
- U1 pad 3: Net-(A1-GPIO10) -> Net-(A1-GPIO2)
- U1 pad 5: +15V -> +15-24V
- U12 pad 2: Net-(A1-GPIO3) -> +15V-24V
- U12 pad 3: Net-(A1-GPIO2) -> GND
- U12 pad 4: Net-(U12-ILIM) -> Net-(J1-Pin_1)
- U2 pad 2: Net-(A1-GPIO13) -> Net-(A1-GPIO7)
- U2 pad 3: Net-(A1-GPIO12) -> Net-(A1-GPIO6)
- U2 pad 5: +15V -> +15-24V
- U3 pad 2: Net-(A1-GPIO15) -> Net-(A1-GPIO9)
- U3 pad 3: Net-(A1-GPIO14) -> Net-(A1-GPIO8)
- U3 pad 5: +15V -> +15-24V
- U4 pad 2: Net-(A1-GPIO9) -> Net-(A1-GPIO11)
- U4 pad 3: Net-(A1-GPIO8) -> Net-(A1-GPIO10)
- U4 pad 5: +15V -> +15-24V
- U5 pad 2: Net-(A1-GPIO28_ADC2) -> Net-(A1-GPIO13)
- U5 pad 3: Net-(A1-GPIO27_ADC1) -> Net-(A1-GPIO12)
- U5 pad 5: +15V -> +15-24V
- U6 pad 2: Net-(A1-GPIO26_ADC0) -> Net-(A1-GPIO15)
- U6 pad 3: Net-(A1-GPIO22) -> Net-(A1-GPIO14)
- U6 pad 5: +15V -> +15-24V
- U7 pad 5: +15V -> +15-24V
- U8 pad 2: +15V-24V -> Net-(A1-GPIO26_ADC0)
- U8 pad 3: GND -> Net-(A1-GPIO22)
- U8 pad 4: Net-(J1-Pin_1) -> Net-(U8-ILIM)
- U9 pad 2: Net-(A1-GPIO7) -> Net-(A1-GPIO28_ADC2)
- U9 pad 3: Net-(A1-GPIO6) -> Net-(A1-GPIO27_ADC1)
- U9 pad 5: +15V -> +15-24V
Routing:
- net +15-24V: track 0.00 -> 185.6 mm, vias 0 -> 44
- net +15V: track 116.2 -> 0.00 mm, vias 1 -> 0
- net Net-(A1-GPIO28_ADC2): track 0.00 -> 77.1 mm
- net Net-(A1-GPIO27_ADC1): track 0.00 -> 71.8 mm, vias 0 -> 2
- net GND: track 208.0 -> 151.9 mm, vias 8 -> 10
- net Net-(A1-GPIO26_ADC0): track 0.00 -> 54.6 mm, vias 0 -> 2
- net Net-(A1-GPIO22): track 0.00 -> 51.7 mm, vias 0 -> 2
- net /Disp_SCL: track 0.00 -> 51.3 mm, vias 0 -> 1
- net Net-(A1-GPIO13): track 0.00 -> 47.6 mm, vias 0 -> 2
- net +3.3V: track 45.4 -> 0.00 mm
- net Net-(A1-GPIO17): track 0.00 -> 40.0 mm, vias 0 -> 2
- net /d_CLK: track 0.00 -> 39.0 mm, vias 0 -> 1
- net +5V: track 37.8 -> 71.1 mm
- net Net-(A1-GPIO16): track 0.00 -> 31.5 mm, vias 0 -> 2
- net Net-(A1-GPIO12): track 19.1 -> 44.1 mm
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Other:
- board size 84.7 x 75 mm -> 80 x 80 mm
- board text added: "26.5 GHz"
- board text added: "Attenuator Controller OE5RNL & OE5NVL V1 202505"
- board text added: "B1"
- board text added: "B2"
- board text added: "B3"
- board text added: "B4"
- board text added: "B5"
- board text added: "B6"
- board text added: "B7"
- board text added: "B8"
- board text added: "B9"
- board text added: "Display"
- board text added: "Drehgeber"

Commit message: .gitignore Schaltung
Parts:
- removed C20: 47uF 50V, Capacitor_SMD:CP_Elec_6.3x5.2
- removed J16: Conn_02x05_Odd_Even, Connector_PinHeader_2.54mm:PinHeader_2x05_P2.54mm_Vertical
- added H1: MountingHole, MountingHole:MountingHole_2.5mm, F.Cu at (56.6, 51.6)
- added H2: MountingHole, MountingHole:MountingHole_2.5mm, F.Cu at (128.6, 51.7)
- added H3: MountingHole, MountingHole:MountingHole_2.5mm, F.Cu at (56.6, 123.5)
- added H4: MountingHole, MountingHole:MountingHole_2.5mm, F.Cu at (128.6, 123.6)
- added J6: Display, Connector_PinHeader_2.54mm:PinHeader_1x04_P2.54mm_Vertical, F.Cu at (128.7, 67.1)
- J2: value Dsiplay -> R&S Attenuator 26.5 GHz; footprint Connector_PinHeader_2.54mm:PinHeader_1x04_P2.54mm_Vertical -> Connector_PinSocket_2.54mm:PinSocket_2x05_P2.54mm_Vertical
- U10: moved to F.Cu
- moved J2 33.8 mm to (126.0, 102.5)
- moved C11 11.9 mm to (101.0, 51.6)
- moved J1 2.20 mm to (120.3, 54.5)
- moved C21 2.20 mm to (107.1, 54.1)
- turned U10 to 180 degrees
Connections:
- J2 pad 1: /D_SDA -> +15V-24V
- J2 pad 2: /Disp_SCL -> /40dBa
- J2 pad 3: +3.3V -> /20dB
- J2 pad 4: GND -> /40dBb
- U1 pad 5: +15-24V -> +15V-24V
- U2 pad 5: +15-24V -> +15V-24V
- U3 pad 5: +15-24V -> +15V-24V
- U4 pad 5: +15-24V -> +15V-24V
- U5 pad 5: +15-24V -> +15V-24V
- U6 pad 5: +15-24V -> +15V-24V
- U7 pad 5: +15-24V -> +15V-24V
- U8 pad 5: +15-24V -> +15V-24V
- U9 pad 5: +15-24V -> +15V-24V
Routing:
- net +15V-24V: track 6.61 -> 269.0 mm, vias 0 -> 61
- net +15-24V: track 185.6 -> 0.00 mm, vias 44 -> 0
- net +3.3V: track 0.00 -> 80.1 mm
- net +5V: track 71.1 -> 121.8 mm
- net /40dBb: track 0.00 -> 46.4 mm
- net /D_SW: track 0.00 -> 42.2 mm, vias 0 -> 1
- net Net-(J1-Pin_1): track 29.9 -> 72.0 mm
- net /D_DT: track 0.00 -> 39.9 mm, vias 0 -> 1
- net /40dBa: track 0.00 -> 22.4 mm, vias 0 -> 1
- net /20dB: track 0.00 -> 12.2 mm
- net GND: track 151.9 -> 161.7 mm, vias 10 -> 9
- net /10dB: track 0.00 -> 7.84 mm
- net /D_SDA: track 50.1 -> 54.4 mm
- net Net-(A1-GPIO26_ADC0): track 54.6 -> 57.9 mm
- net Net-(A1-GPIO11): track 47.1 -> 50.4 mm
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Other:
- board text added: "Attenuator Controller OE5RNL&OE5NVL V1 202505"
- board text removed: "Attenuator Controller OE5RNL & OE5NVL V1 202505"

Commit message: R umbenannt. div bereinigungen
Parts:
- renumbered C9 to C1, C8 to C2, C4 to C3, C1 to C4, C2 to C5, C3 to C6, C6 to C8, C5 to C9, R9 to R1, R8 to R2, R4 to R3, R1 to R4, R2 to R5, R3 to R6, R6 to R8, R5 to R9
Routing:
- net +15V-24V: vias 61 -> 69
Other:
- board text added: "+12V"
- board text added: "+15-24V"
- board text added: "+5V"
- board text added: "ESP-Display"
- board text added: "H-Brides"
- board text added: "PICO-Display"
- board text added: "U12"
- board text removed: "Display"
