File: Schaltung/att.kicad_pcb (KiCad board)
At the start: 2 copper layers, 80 x 80 mm, 48 parts, among them J1 12V Power supply, J2 R&S Attenuator 26.5 GHz, J3 dB Drehgeber, J4 ESP-Controller, J6 Display, U1 DRV8871DDA, U2 DRV8871DDA, U3 DRV8871DDA, U4 DRV8871DDA, U5 DRV8871DDA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

Commit message: Version 1.1 der Schaltung
Parts:
- added J5: xxx, 0_RNL_ATT:PinHeader_2x02_P2.54mm_Vertical, F.Cu at (126.2, 66.1)
- moved R11 2.82 mm to (127.6, 59.9)
- moved R10 2.54 mm to (127.6, 56.7)
- moved J6 2.02 mm to (128.8, 79.8)
- moved U11 0.10 mm to (111.5, 88.5)
Routing:
- net Net-(J1-Pin_1): track 85.9 -> 104.2 mm
- net +15V-24V: track 250.6 -> 246.1 mm
- net +3.3V: track 102.4 -> 106.4 mm
- net Net-(A1-GPIO26_ADC0): track 50.6 -> 53.4 mm, vias 2 -> 1
- net Net-(A1-GPIO11): track 48.8 -> 46.4 mm
- net Net-(U13I-B9b): track 11.5 -> 13.8 mm
- net /40dBb: track 30.0 -> 28.3 mm
- net Net-(A1-GPIO13): track 46.4 -> 44.9 mm
- net Net-(A1-GPIO10): track 48.9 -> 47.4 mm
- net Net-(A1-GPIO12): track 42.6 -> 41.1 mm
- net /10dB: track 21.5 -> 20.2 mm
- net +5V: track 108.9 -> 110.2 mm
- net /D_SW: track 54.4 -> 53.3 mm
- net /D_SDA: track 54.4 -> 55.4 mm
- net /Disp_SCL: track 54.3 -> 55.2 mm
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Other:
- board text added: "3,3V"
- board text added: "CLK"
- board text added: "DT"
- board text added: "D_SW"
- board text added: "GND"
- board text added: "OE5RNL&OE5NVL Attenuator-Controller V1.1 202604 ADL516"
- board text added: "RX"
- board text added: "SCL"
- board text added: "SDA"
- board text added: "TX"
- board text removed: "OE5RNL&OE5NVL Attenuator-Controller V1.0 202604 ADL516"
