File: Schaltung/att.kicad_sch (KiCad schematic)
At the start: 52 parts, among them J1 12V Power supply, J10 RF_ON_OFF, J11 40dB_B, J12 10dB, J15 5V für ESP Panel, J16 Conn_02x05_Odd_Even, J17 20dB_A, J18 20dB_A, J2 Dsiplay, J3 dB Drehgeber, J4 ESP-Controller, J5 ATT_SEL, J6 20dB_A, J7 40dB_A, J8 20dB_B, J9 5dB, U1 DRV8871DDA, U12 DRV8871DDA, U2 DRV8871DDA, U3 DRV8871DDA, U4 DRV8871DDA, U5 DRV8871DDA, U6 DRV8871DDA, U7 DRV8871DDA, U9 DRV8871DDA

Commit message: schaltung PCB
Parts:
- removed J10: RF_ON_OFF, Connector_PinHeader_2.54mm:PinHeader_1x02_P2.54mm_Vertical, symbol Connector:Conn_01x02_Pin
- removed J11: 40dB_B, Connector_PinHeader_2.54mm:PinHeader_1x02_P2.54mm_Vertical, symbol Connector:Conn_01x02_Pin
- removed J12: 10dB, Connector_PinHeader_2.54mm:PinHeader_1x02_P2.54mm_Vertical, symbol Connector:Conn_01x02_Pin
- removed J15: 5V für ESP Panel, Connector_PinHeader_2.54mm:PinHeader_1x02_P2.54mm_Vertical, symbol Connector:Conn_01x02_Pin
- removed J17, J18, J6: 20dB_A, Connector_PinHeader_2.54mm:PinHeader_1x02_P2.54mm_Vertical, symbol Connector:Conn_01x02_Pin
- removed J4: ESP-Controller, Connector_PinHeader_2.54mm:PinHeader_1x03_P2.54mm_Vertical, symbol Connector:Conn_01x03_Pin
- removed J7: 40dB_A, Connector_PinHeader_2.54mm:PinHeader_1x02_P2.54mm_Vertical, symbol Connector:Conn_01x02_Pin
- removed J8: 20dB_B, Connector_PinHeader_2.54mm:PinHeader_1x02_P2.54mm_Vertical, symbol Connector:Conn_01x02_Pin
- removed J9: 5dB, Connector_PinHeader_2.54mm:PinHeader_1x02_P2.54mm_Vertical, symbol Connector:Conn_01x02_Pin
- added J4: ESP-Controller, Connector_PinHeader_2.54mm:PinHeader_1x04_P2.54mm_Vertical, symbol Connector:Conn_01x04_Pin
- added U13: (no value), 0_RNL_ATT:SIL_18, symbol 0_RNL_ATT:con-1-18-unabhängig
- C4: footprint Capacitor_SMD:C_0805_2012Metric_Pad1.18x1.45mm_HandSolder -> Resistor_SMD:R_0805_2012Metric
- R1, R4, R8, R9: footprint Resistor_SMD:R_0805_2012Metric_Pad1.20x1.40mm_HandSolder -> Resistor_SMD:R_0805_2012Metric
- renumbered U12 to U1, U8 to U12, U9 to U2, U4 to U3, U1 to U4, U2 to U5, U3 to U6, U6 to U8, U5 to U9
Connections:
- net +15V: no longer U1.5 (VM), U2.5 (VM), U3.5 (VM), U4.5 (VM), U5.5 (VM), U6.5 (VM), U7.5 (VM), U8.5 (VM), U9.5 (VM)
- net +15V-24V: no longer C20.1
- net +5V: now also J4.1 (Pin_1)
- net GND: now also J4.4 (Pin_4); no longer C20.2
- net at U7.6 (OUT1): now also U13.13 (B7a)
- net at U7.8 (OUT2): now also U13.14 (B7b)
- net TX: now reaches A1.1 (GPIO0)
- net TX: now also J4.2 (Pin_2)
- net RX: now reaches A1.2 (GPIO1)
- net RX: now also J4.3 (Pin_3)
- net at U1.6 (OUT1): now also U13.1 (B1a)
- net at U1.8 (OUT2): now also U13.2 (B1b)
- net at U2.6 (OUT1): now also U13.3 (B2a)
- net at U2.8 (OUT2): now also U13.4 (B2b)
- net at U6.8 (OUT2): now also U13.12 (B6b)
- net at U6.6 (OUT1): now also U13.11 (B6a)
- net at U9.8 (OUT2): now also U13.18 (B9b)
- net at U9.6 (OUT1): now also U13.17 (B9a)
- net at U5.6 (OUT1): now also U13.9 (B5a)
- net at U5.8 (OUT2): now also U13.10 (B5b)
- net at U3.6 (OUT1): now also U13.5 (B3a)
- net at U3.8 (OUT2): now also U13.6 (B3b)
- net at U4.6 (OUT1): now also U13.7 (B4a)
- net at U4.8 (OUT2): now also U13.8 (B4b)
- net at U8.6 (OUT1): now also U13.15 (B8a)
- net at U8.8 (OUT2): now also U13.16 (B8b)
- new net +15-24V: U1.5 (VM), U2.5 (VM), U3.5 (VM), U4.5 (VM), U5.5 (VM), U6.5 (VM), U7.5 (VM), U8.5 (VM), U9.5 (VM)
Other:
- note removed: "GND"
- note removed: "RXD"
- note removed: "TXD"
- moved on the sheet: C20

Commit message: .gitignore Schaltung
Parts:
- removed C20: 47uF 50V, Capacitor_SMD:CP_Elec_6.3x5.2, symbol Device:C_Polarized
- removed J16: Conn_02x05_Odd_Even, Connector_PinHeader_2.54mm:PinHeader_2x05_P2.54mm_Vertical, symbol Connector_Generic:Conn_02x05_Odd_Even
- removed J2: Dsiplay, Connector_PinHeader_2.54mm:PinHeader_1x04_P2.54mm_Vertical, symbol Connector:Conn_01x04_Pin
- added H1, H2, H3, H4: MountingHole, MountingHole:MountingHole_2.5mm, symbol Mechanical:MountingHole
- added J2: R&S Attenuator 26.5 GHz, Connector_PinSocket_2.54mm:PinSocket_2x05_P2.54mm_Vertical, symbol 0_RNL_ATT:Conn_02x05_26GHz_Att
- added J6: Display, Connector_PinHeader_2.54mm:PinHeader_1x04_P2.54mm_Vertical, symbol Connector:Conn_01x04_Pin
Connections:
- net +15-24V is gone; now on net +15V-24V: U1.5 (VM), U2.5 (VM), U3.5 (VM), U4.5 (VM), U5.5 (VM), U6.5 (VM), U7.5 (VM), U8.5 (VM), U9.5 (VM)
- net +15V-24V: now also J2.1 (Pin_10)
- net +3.3V: now also J6.2 (Pin_2)
- net 10dB: now also J2.9 (Pin_6)
- net 20dB: now also J2.3 (Pin_9)
- net 40dBa: now also J2.2 (Pin_1)
- net 40dBb: now also J2.4 (Pin_2)
- net D_SDA: now also J6.4 (Pin_4)
- net Disp_SCL: now also J6.3 (Pin_3)
- net GND: now also J2.7 (Pin_7), J2.8 (Pin_4), J6.1 (Pin_1)

Commit message: R umbenannt. div bereinigungen
Parts:
- renumbered C9 to C1, C8 to C2, C4 to C3, C1 to C4, C2 to C5, C3 to C6, C6 to C8, C5 to C9, R9 to R1, R8 to R2, R4 to R3, R1 to R4, R2 to R5, R3 to R6, R6 to R8, R5 to R9
Other:
- moved on the sheet: H1, H2, H3, H4
Changed lines of the file:
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@@
 		(in_pos_files yes)
 		(dnp no)
-		(property "Reference" "R5"
+		(property "Reference" "R9"
 			(at 206.502 143.256 90)
 			(show_name no)
@@
 			(project "att"
 				(path "/018aec4b-c766-4652-8f21-caeb401652b2"
-					(reference "R5")
+					(reference "R9")
 					(unit 1)
 				)
@@
 		(in_pos_files yes)
 		(dnp no)
-		(property "Reference" "R2"
+		(property "Reference" "R5"
 			(at 34.798 177.292 90)
 			(show_name no)
@@
 			(project "att"
 				(path "/018aec4b-c766-4652-8f21-caeb401652b2"
-					(reference "R2")
+					(reference "R5")
 					(unit 1)
 				)
@@
 		(in_pos_files yes)
 		(dnp no)
-		(property "Reference" "C5"
+		(property "Reference" "C9"
 			(at 204.724 152.654 90)
 			(show_name no)
@@
 			(project "att"
 				(path "/018aec4b-c766-4652-8f21-caeb401652b2"
-					(reference "C5")
+					(reference "C9")
 					(unit 1)
 				)
@@
 		(in_pos_files yes)
 		(dnp no)
-		(property "Reference" "R3"
+		(property "Reference" "R6"
 			(at 147.066 155.956 90)
 			(show_name no)
@@
 			(project "att"
 				(path "/018aec4b-c766-4652-8f21-caeb401652b2"
-					(reference "R3")
+					(reference "R6")
 					(unit 1)
 				)
@@
 		(in_pos_files yes)
 		(dnp no)
-		(property "Reference" "C4"
+		(property "Reference" "C3"
 			(at 145.034 194.056 90)
 			(show_name no)
@@
 			(project "att"
 				(path "/018aec4b-c766-4652-8f21-caeb401652b2"
-					(reference "C4")
+					(reference "C3")
 					(unit 1)
 				)
@@
 	(symbol
 		(lib_id "Mechanical:MountingHole")
-		(at 255.27 156.21 0)
+		(at 257.81 161.29 0)
 		(unit 1)
 		(body_style 1)
@@
 		(fields_autoplaced yes)
 		(property "Reference" "H2"
-			(at 257.81 154.9399 0)
+			(at 260.35 160.0199 0)
 			(show_name no)
 			(do_not_autoplace no)
@@
 		)
 		(property "Value" "MountingHole"
-			(at 257.81 157.4799 0)
+			(at 260.35 162.5599 0)
+			(hide yes)
 			(show_name no)
 			(do_not_autoplace no)
@@
 		)
 		(property "Footprint" "MountingHole:MountingHole_2.5mm"
-			(at 255.27 156.21 0)
+			(at 257.81 161.29 0)
 			(hide yes)
 			(show_name no)
@@
 		)
 		(property "Datasheet" ""
-			(at 255.27 156.21 0)
+			(at 257.81 161.29 0)
 			(hide yes)
 			(show_name no)
@@
 		)
 		(property "Description" "Mounting Hole without connection"
-			(at 255.27 156.21 0)
+			(at 257.81 161.29 0)
 			(hide yes)
 			(show_name no)
@@
 		(in_pos_files yes)
 		(dnp no)
-		(property "Reference" "R9"
+		(property "Reference" "R1"
 			(at 75.692 59.69 90)
 			(show_name no)
@@
 			(project "att"
 				(path "/018aec4b-c766-4652-8f21-caeb401652b2"
-					(reference "R9")
+					(reference "R1")
 					(unit 1)
 				)
@@
 		(in_pos_files yes)
 		(dnp no)
-		(property "Reference" "R4"
+		(property "Reference" "R3"
 			(at 146.812 183.642 90)
 			(show_name no)
@@
 			(project "att"
 				(path "/018aec4b-c766-4652-8f21-caeb401652b2"
-					(reference "R4")
+					(reference "R3")
 					(unit 1)
 				)
@@
 	(symbol
 		(lib_id "Mechanical:MountingHole")
-		(at 266.7 152.4 0)
+		(at 275.59 161.29 0)
 		(unit 1)
 		(body_style 1)
@@
 		(fields_autoplaced yes)
 		(property "Reference" "H4"
-			(at 269.24 151.1299 0)
+			(at 278.13 160.0199 0)
 			(show_name no)
 			(do_not_autoplace no)
@@
 		)
 		(property "Value" "MountingHole"
-			(at 269.24 153.6699 0)
+			(at 278.13 162.5599 0)
+			(hide yes)
 			(show_name no)
 			(do_not_autoplace no)
@@
 		)
 		(property "Footprint" "MountingHole:MountingHole_2.5mm"
-			(at 266.7 152.4 0)
+			(at 275.59 161.29 0)
 			(hide yes)
 			(show_name no)
@@
 		)
 		(property "Datasheet" ""
-			(at 266.7 152.4 0)
+			(at 275.59 161.29 0)
 			(hide yes)
 			(show_name no)
@@
 		)
 		(property "Description" "Mounting Hole without connection"
-			(at 266.7 152.4 0)
+			(at 275.59 161.29 0)
 			(hide yes)
 			(show_name no)
@@
 		(in_pos_files yes)
 		(dnp no)
-		(property "Reference" "R8"
+		(property "Reference" "R2"
 			(at 31.242 59.69 90)
 			(show_name no)
@@
 			(project "att"
 				(path "/018aec4b-c766-4652-8f21-caeb401652b2"
-					(reference "R8")
+					(reference "R2")
 					(unit 1)
 				)
@@
 	(symbol
 		(lib_id "Mechanical:MountingHole")
-		(at 259.08 147.32 0)
+		(at 266.7 161.29 0)
 		(unit 1)
 		(body_style 1)
@@
 		(fields_autoplaced yes)
 		(property "Reference" "H3"
-			(at 261.62 146.0499 0)
+			(at 269.24 160.0199 0)
 			(show_name no)
 			(do_not_autoplace no)
@@
 		)
 		(property "Value" "MountingHole"
-			(at 261.62 148.5899 0)
+			(at 269.24 162.5599 0)
+			(hide yes)
 			(show_name no)
 			(do_not_autoplace no)
@@
 		)
 		(property "Footprint" "MountingHole:MountingHole_2.5mm"
-			(at 259.08 147.32 0)
+			(at 266.7 161.29 0)
 			(hide yes)
 			(show_name no)
@@
 		)
 		(property "Datasheet" ""
-			(at 259.08 147.32 0)
+			(at 266.7 161.29 0)
 			(hide yes)
 			(show_name no)
@@
 		)
 		(property "Description" "Mounting Hole without connection"
-			(at 259.08 147.32 0)
+			(at 266.7 161.29 0)
 			(hide yes)
 			(show_name no)
@@
 		(in_pos_files yes)
 		(dnp no)
-		(property "Reference" "C1"
+		(property "Reference" "C4"
 			(at 34.036 161.798 90)
 			(show_name no)
@@
 			(project "att"
 				(path "/018aec4b-c766-4652-8f21-caeb401652b2"
-					(reference "C1")
+					(reference "C4")
 					(unit 1)
 				)
@@
 		(in_pos_files yes)
 		(dnp no)
-		(property "Reference" "C3"
+		(property "Reference" "C6"
 			(at 144.78 166.624 90)
 			(show_name no)
@@
 			(project "att"
 				(path "/018aec4b-c766-4652-8f21-caeb401652b2"
-					(reference "C3")
+					(reference "C6")
 					(unit 1)
 				)
@@
 		(in_pos_files yes)
 		(dnp no)
-		(property "Reference" "C2"
+		(property "Reference" "C5"
 			(at 33.528 189.23 90)
 			(show_name no)
@@
 			(project "att"
 				(path "/018aec4b-c766-4652-8f21-caeb401652b2"
-					(reference "C2")
+					(reference "C5")
 					(unit 1)
 				)
@@
 		(in_pos_files yes)
 		(dnp no)
-		(property "Reference" "C9"
+		(property "Reference" "C1"
 			(at 74.676 71.628 90)
 			(show_name no)
@@
 			(project "att"
 				(path "/018aec4b-c766-4652-8f21-caeb401652b2"
-					(reference "C9")
+					(reference "C1")
 					(unit 1)
 				)
@@
 	(symbol
 		(lib_id "Mechanical:MountingHole")
-		(at 246.38 149.86 0)
+		(at 248.92 161.29 0)
 		(unit 1)
 		(body_style 1)
@@
 		(fields_autoplaced yes)
 		(property "Reference" "H1"
-			(at 248.92 148.5899 0)
+			(at 251.46 160.0199 0)
 			(show_name no)
 			(do_not_autoplace no)
@@
 		)
 		(property "Value" "MountingHole"
-			(at 248.92 151.1299 0)
+			(at 251.46 162.5599 0)
+			(hide yes)
 			(show_name no)
 			(do_not_autoplace no)
@@
 		)
 		(property "Footprint" "MountingHole:MountingHole_2.5mm"
-			(at 246.38 149.86 0)
+			(at 248.92 161.29 0)
 			(hide yes)
 			(show_name no)
@@
 		)
 		(property "Datasheet" ""
-			(at 246.38 149.86 0)
+			(at 248.92 161.29 0)
 			(hide yes)
 			(show_name no)
@@
 		)
 		(property "Description" "Mounting Hole without connection"
-			(at 246.38 149.86 0)
+			(at 248.92 161.29 0)
 			(hide yes)
 			(show_name no)
@@
 		(in_pos_files yes)
 		(dnp no)
-		(property "Reference" "R6"
+		(property "Reference" "R8"
 			(at 206.502 115.062 90)
 			(show_name no)
@@
 			(project "att"
 				(path "/018aec4b-c766-4652-8f21-caeb401652b2"
-					(reference "R6")
+					(reference "R8")
 					(unit 1)
 				)
@@
 		(in_pos_files yes)
 		(dnp no)
-		(property "Reference" "C6"
+		(property "Reference" "C8"
 			(at 204.978 125.476 90)
 			(show_name no)
@@
 			(project "att"
 				(path "/018aec4b-c766-4652-8f21-caeb401652b2"
-					(reference "C6")
+					(reference "C8")
 					(unit 1)
 				)
@@
 		(in_pos_files yes)
 		(dnp no)
-		(property "Reference" "R1"
+		(property "Reference" "R4"
 			(at 35.052 149.86 90)
 			(show_name no)
@@
 			(project "att"
 				(path "/018aec4b-c766-4652-8f21-caeb401652b2"
-					(reference "R1")
+					(reference "R4")
 					(unit 1)
 				)
@@
 		(in_pos_files yes)
 		(dnp no)
-		(property "Reference" "C8"
+		(property "Reference" "C2"
 			(at 30.226 71.628 90)
 			(show_name no)
@@
 			(project "att"
 				(path "/018aec4b-c766-4652-8f21-caeb401652b2"
-					(reference "C8")
+					(reference "C2")
 					(unit 1)
 				)

Commit message: produktion
Parts:
- J2: footprint Connector_PinSocket_2.54mm:PinSocket_2x05_P2.54mm_Vertical -> Connector_PinHeader_2.54mm:PinHeader_2x05_P2.54mm_Vertical
- J5: footprint (none) -> Connector_PinSocket_2.54mm:PinSocket_2x02_P2.54mm_Vertical
Connections:
- net +15V-24V: now also J2.2 (Pin_10); no longer J2.1 (Pin_10)
- net 10dB: now also J2.10 (Pin_6); no longer J2.9 (Pin_6)
- net 20dB: now also J2.4 (Pin_9); no longer J2.3 (Pin_9)
- net 40dBa: now also J2.1 (Pin_1); no longer J2.2 (Pin_1)
- net 40dBb: now also J2.3 (Pin_2); no longer J2.4 (Pin_2)
- net at A1.4 (GPIO2), U1.3 (IN1): now also J5.3 (Pin_3); no longer J5.1 (Pin_1)
- net at A1.5 (GPIO3), U1.2 (IN2): now also J5.1 (Pin_1); no longer J5.3 (Pin_3)
Changed lines of the file:
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@@
 	)
 	(junction
-		(at 41.91 180.34)
+		(at 128.27 54.61)
 		(diameter 0)
 		(color 0 0 0 0)
 	)
 	(junction
-		(at 86.36 107.95)
+		(at 41.91 180.34)
 		(diameter 0)
 		(color 0 0 0 0)
 	)
 	(junction
-		(at 107.95 54.61)
+		(at 86.36 107.95)
 		(diameter 0)
 		(color 0 0 0 0)
@@
 	)
 	(junction
-		(at 128.27 54.61)
+		(at 107.95 54.61)
 		(diameter 0)
 		(color 0 0 0 0)
@@
 	)
 	(junction
-		(at 250.19 41.91)
+		(at 110.49 52.07)
 		(diameter 0)
 		(color 0 0 0 0)
 	)
 	(junction
-		(at 110.49 52.07)
+		(at 250.19 41.91)
 		(diameter 0)
 		(color 0 0 0 0)
@@
 	(wire
 		(pts
+			(xy 127 52.07) (xy 128.27 52.07)
+		)
+		(stroke
+			(width 0)
+			(type default)
+		)
+	)
+	(wire
+		(pts
 			(xy 62.23 76.2) (xy 102.87 76.2)
 		)
@@
 	(wire
 		(pts
+			(xy 127 54.61) (xy 128.27 54.61)
+		)
+		(stroke
+			(width 0)
+			(type default)
+		)
+	)
+	(wire
+		(pts
 			(xy 204.47 41.91) (xy 204.47 43.18)
 		)
@@
 	(wire
 		(pts
-			(xy 110.49 52.07) (xy 114.3 52.07)
-		)
-		(stroke
-			(width 0)
-			(type default)
-		)
-	)
-	(wire
-		(pts
 			(xy 152.4 158.75) (xy 153.67 158.75)
 		)
@@
 	(wire
 		(pts
-			(xy 107.95 54.61) (xy 114.3 54.61)
+			(xy 26.67 67.31) (xy 29.21 67.31)
 		)
 		(stroke
@@
 	(wire
 		(pts
-			(xy 26.67 67.31) (xy 29.21 67.31)
+			(xy 62.23 54.61) (xy 62.23 76.2)
 		)
 		(stroke
@@
 	(wire
 		(pts
-			(xy 62.23 54.61) (xy 62.23 76.2)
+			(xy 40.64 85.09) (xy 115.57 85.09)
 		)
 		(stroke
@@
 	(wire
 		(pts
-			(xy 40.64 85.09) (xy 115.57 85.09)
+			(xy 115.57 120.65) (xy 106.68 120.65)
 		)
 		(stroke
@@
 	(wire
 		(pts
-			(xy 115.57 120.65) (xy 106.68 120.65)
+			(xy 63.5 144.78) (xy 88.9 144.78)
 		)
 		(stroke
@@
 	(wire
 		(pts
-			(xy 63.5 144.78) (xy 88.9 144.78)
+			(xy 49.53 21.59) (xy 49.53 26.67)
 		)
 		(stroke
@@
 	(wire
 		(pts
-			(xy 49.53 21.59) (xy 49.53 26.67)
+			(xy 128.27 52.07) (xy 128.27 54.61)
 		)
 		(stroke
@@
 	(wire
 		(pts
-			(xy 127 52.07) (xy 128.27 52.07)
-		)
-		(stroke
-			(width 0)
-			(type default)
-		)
-	)
-	(wire
-		(pts
 			(xy 161.29 110.49) (xy 181.61 110.49)
 		)
@@
 	(wire
 		(pts
+			(xy 110.49 52.07) (xy 114.3 52.07)
+		)
+		(stroke
+			(width 0)
+			(type default)
+		)
+	)
+	(wire
+		(pts
 			(xy 104.14 52.07) (xy 110.49 52.07)
 		)
@@
 	(wire
 		(pts
-			(xy 57.15 110.49) (xy 64.77 110.49)
+			(xy 107.95 54.61) (xy 114.3 54.61)
 		)
 		(stroke
@@
 	(wire
 		(pts
-			(xy 260.35 41.91) (xy 262.89 41.91)
+			(xy 57.15 110.49) (xy 64.77 110.49)
 		)
 		(stroke
@@
 	(wire
 		(pts
-			(xy 227.33 39.37) (xy 227.33 41.91)
+			(xy 260.35 41.91) (xy 262.89 41.91)
 		)
 		(stroke
@@
 	(wire
 		(pts
-			(xy 201.93 67.31) (xy 209.55 67.31)
+			(xy 227.33 39.37) (xy 227.33 41.91)
 		)
 		(stroke
@@
 	(wire
 		(pts
-			(xy 143.51 54.61) (xy 143.51 59.69)
+			(xy 201.93 67.31) (xy 209.55 67.31)
 		)
 		(stroke
@@
 	(wire
 		(pts
-			(xy 250.19 39.37) (xy 250.19 41.91)
+			(xy 143.51 54.61) (xy 143.51 59.69)
 		)
 		(stroke
@@
 	(wire
 		(pts
-			(xy 127 54.61) (xy 128.27 54.61)
+			(xy 250.19 39.37) (xy 250.19 41.91)
 		)
 		(stroke
@@
 	(wire
 		(pts
-			(xy 128.27 52.07) (xy 128.27 54.61)
-		)
-		(stroke
-			(width 0)
-			(type default)
-		)
-	)
-	(wire
-		(pts
 			(xy 212.09 151.13) (xy 214.63 151.13)
 		)
@@
 		(in_pos_files yes)
 		(dnp no)
-		(fields_autoplaced yes)
 		(property "Reference" "J2"
 			(at 36.83 99.06 0)
@@
 		)
 		(property "Value" "R&S Attenuator 26.5 GHz"
-			(at 36.83 101.6 0)
+			(at 38.354 122.936 0)
 			(show_name no)
 			(do_not_autoplace no)
@@
 			)
 		)
-		(property "Footprint" "Connector_PinSocket_2.54mm:PinSocket_2x05_P2.54mm_Vertical"
+		(property "Footprint" "Connector_PinHeader_2.54mm:PinHeader_2x05_P2.54mm_Vertical"
 			(at 38.1 110.49 0)
 			(hide yes)
@@
 	(symbol
 		(lib_id "Connector_Generic:Conn_02x02_Odd_Even")
-		(at 119.38 52.07 0)
+		(at 119.38 54.61 0)
+		(mirror x)
 		(unit 1)
 		(body_style 1)
@@
 		(dnp no)
 		(property "Reference" "J5"
-			(at 114.554 48.514 0)
+			(at 114.554 58.166 0)
 			(show_name no)
 			(do_not_autoplace no)
@@
 		)
 		(property "Value" "ATT_SEL"
-			(at 120.65 48.26 0)
+			(at 120.65 58.42 0)
 			(show_name no)
 			(do_not_autoplace no)
@@
 			)
 		)
-		(property "Footprint" ""
-			(at 119.38 52.07 0)
+		(property "Footprint" "Connector_PinSocket_2.54mm:PinSocket_2x02_P2.54mm_Vertical"
+			(at 119.38 54.61 0)
 			(hide yes)
 			(show_name no)
@@
 		)
 		(property "Datasheet" ""
-			(at 119.38 52.07 0)
+			(at 119.38 54.61 0)
 			(hide yes)
 			(show_name no)
@@
 		)
 		(property "Description" "Generic connector, double row, 02x02, odd/even pin numbering scheme (row 1 odd numbers, row 2 even numbers), script generated (kicad-library-utils/schlib/autogen/connector/)"
-			(at 119.38 52.07 0)
+			(at 119.38 54.61 0)
 			(hide yes)
 			(show_name no)

Commit message: production-files
Parts:
- J5: footprint Connector_PinSocket_2.54mm:PinSocket_2x02_P2.54mm_Vertical -> Connector_PinHeader_2.54mm:PinHeader_2x02_P2.54mm_Vertical
Connections:
- net at A1.5 (GPIO3), U1.2 (IN2): now also J5.3 (Pin_3); no longer J5.1 (Pin_1)
- net at A1.4 (GPIO2), U1.3 (IN1): now also J5.1 (Pin_1); no longer J5.3 (Pin_3)
Changed lines of the file:
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@@
 	)
 	(junction
-		(at 128.27 54.61)
-		(diameter 0)
-		(color 0 0 0 0)
-	)
-	(junction
 		(at 41.91 180.34)
 		(diameter 0)
@@
 	)
 	(junction
-		(at 41.91 152.4)
+		(at 107.95 54.61)
 		(diameter 0)
 		(color 0 0 0 0)
 	)
 	(junction
-		(at 107.95 54.61)
+		(at 41.91 152.4)
 		(diameter 0)
 		(color 0 0 0 0)
@@
 	)
 	(junction
+		(at 128.27 54.61)
+		(diameter 0)
+		(color 0 0 0 0)
+	)
+	(junction
 		(at 143.51 186.69)
 		(diameter 0)
@@
 	(wire
 		(pts
+			(xy 128.27 52.07) (xy 128.27 54.61)
+		)
+		(stroke
+			(width 0)
+			(type default)
+		)
+	)
+	(wire
+		(pts
 			(xy 152.4 186.69) (xy 153.67 186.69)
 		)
@@
 	(wire
 		(pts
-			(xy 260.35 44.45) (xy 260.35 48.26)
+			(xy 107.95 54.61) (xy 107.95 90.17)
 		)
 		(stroke
@@
 	(wire
 		(pts
-			(xy 201.93 146.05) (xy 203.2 146.05)
+			(xy 260.35 44.45) (xy 260.35 48.26)
 		)
 		(stroke
@@
 	(wire
 		(pts
-			(xy 27.94 118.11) (xy 27.94 115.57)
+			(xy 201.93 146.05) (xy 203.2 146.05)
 		)
 		(stroke
@@
 	(wire
 		(pts
-			(xy 127 52.07) (xy 128.27 52.07)
+			(xy 27.94 118.11) (xy 27.94 115.57)
 		)
 		(stroke
@@
 	(wire
 		(pts
-			(xy 62.23 76.2) (xy 102.87 76.2)
+			(xy 127 52.07) (xy 128.27 52.07)
 		)
 		(stroke
@@
 	(wire
 		(pts
-			(xy 161.29 92.71) (xy 259.08 92.71)
+			(xy 62.23 76.2) (xy 102.87 76.2)
 		)
 		(stroke
@@
 	(wire
 		(pts
-			(xy 80.01 102.87) (xy 81.28 102.87)
+			(xy 161.29 92.71) (xy 259.08 92.71)
 		)
 		(stroke
@@
 	(wire
 		(pts
-			(xy 128.27 54.61) (xy 128.27 57.15)
+			(xy 127 54.61) (xy 128.27 54.61)
 		)
 		(stroke
@@
 	(wire
 		(pts
-			(xy 127 54.61) (xy 128.27 54.61)
+			(xy 80.01 102.87) (xy 81.28 102.87)
 		)
 		(stroke
@@
 	(wire
 		(pts
-			(xy 128.27 52.07) (xy 128.27 54.61)
-		)
-		(stroke
-			(width 0)
-			(type default)
-		)
-	)
-	(wire
-		(pts
 			(xy 247.65 41.91) (xy 250.19 41.91)
 		)
@@
 	(wire
 		(pts
+			(xy 128.27 54.61) (xy 128.27 57.15)
+		)
+		(stroke
+			(width 0)
+			(type default)
+		)
+	)
+	(wire
+		(pts
 			(xy 167.64 67.31) (xy 181.61 67.31)
 		)
@@
 	(wire
 		(pts
-			(xy 107.95 54.61) (xy 114.3 54.61)
-		)
-		(stroke
-			(width 0)
-			(type default)
-		)
-	)
-	(wire
-		(pts
 			(xy 57.15 110.49) (xy 64.77 110.49)
 		)
@@
 	(wire
 		(pts
+			(xy 107.95 54.61) (xy 114.3 54.61)
+		)
+		(stroke
+			(width 0)
+			(type default)
+		)
+	)
+	(wire
+		(pts
 			(xy 30.48 185.42) (xy 33.02 185.42)
 		)
@@
 	(wire
 		(pts
-			(xy 107.95 54.61) (xy 107.95 90.17)
-		)
-		(stroke
-			(width 0)
-			(type default)
-		)
-	)
-	(wire
-		(pts
 			(xy 250.19 48.26) (xy 260.35 48.26)
 		)
@@
 	(symbol
 		(lib_id "Connector_Generic:Conn_02x02_Odd_Even")
-		(at 119.38 54.61 0)
-		(mirror x)
+		(at 119.38 52.07 0)
 		(unit 1)
 		(body_style 1)
@@
 		(dnp no)
 		(property "Reference" "J5"
-			(at 114.554 58.166 0)
+			(at 114.554 48.514 0)
 			(show_name no)
 			(do_not_autoplace no)
@@
 		)
 		(property "Value" "ATT_SEL"
-			(at 120.65 58.42 0)
+			(at 120.65 48.26 0)
 			(show_name no)
 			(do_not_autoplace no)
@@
 			)
 		)
-		(property "Footprint" "Connector_PinSocket_2.54mm:PinSocket_2x02_P2.54mm_Vertical"
-			(at 119.38 54.61 0)
+		(property "Footprint" "Connector_PinHeader_2.54mm:PinHeader_2x02_P2.54mm_Vertical"
+			(at 119.38 52.07 0)
 			(hide yes)
 			(show_name no)
@@
 		)
 		(property "Datasheet" ""
-			(at 119.38 54.61 0)
+			(at 119.38 52.07 0)
 			(hide yes)
 			(show_name no)
@@
 		)
 		(property "Description" "Generic connector, double row, 02x02, odd/even pin numbering scheme (row 1 odd numbers, row 2 even numbers), script generated (kicad-library-utils/schlib/autogen/connector/)"
-			(at 119.38 54.61 0)
+			(at 119.38 52.07 0)
 			(hide yes)
 			(show_name no)

Commit message: final vor nvl check
Parts:
- C10: footprint Capacitor_SMD:CP_Elec_6.3x5.2 -> Capacitor_THT:CP_Radial_D8.0mm_P5.00mm
Changed lines of the file:
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@@
 			)
 		)
-		(property "Footprint" "Capacitor_SMD:CP_Elec_6.3x5.2"
+		(property "Footprint" "Capacitor_THT:CP_Radial_D8.0mm_P5.00mm"
 			(at 50.4952 34.29 0)
 			(hide yes)
