File: Schaltung/att.kicad_sch (KiCad schematic)
At the start: 46 parts, among them J1 12V Power supply, J2 R&S Attenuator 26.5 GHz, J3 dB Drehgeber, J4 ESP-Controller, J5 ATT_SEL, J6 Display, U1 DRV8871DDA, U2 DRV8871DDA, U3 DRV8871DDA, U4 DRV8871DDA, U5 DRV8871DDA, U6 DRV8871DDA, U7 DRV8871DDA, U8 DRV8871DDA, U9 DRV8871DDA

Commit message: Stückliste
Parts:
- C1, C2, C3, C4: footprint Resistor_SMD:R_0805_2012Metric -> Capacitor_SMD:C_0805_2012Metric_Pad1.18x1.45mm_HandSolder
Changed lines of the file:
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@@
 			)
 		)
-		(property "Footprint" "Resistor_SMD:R_0805_2012Metric"
+		(property "Footprint" "Capacitor_SMD:C_0805_2012Metric_Pad1.18x1.45mm_HandSolder"
 			(at 152.4 190.8048 0)
 			(hide yes)
@@
 			)
 		)
-		(property "Footprint" "Resistor_SMD:R_0805_2012Metric"
+		(property "Footprint" "Capacitor_SMD:C_0805_2012Metric_Pad1.18x1.45mm_HandSolder"
 			(at 40.64 156.5148 0)
 			(hide yes)
@@
 			)
 		)
-		(property "Footprint" "Resistor_SMD:R_0805_2012Metric"
+		(property "Footprint" "Capacitor_SMD:C_0805_2012Metric_Pad1.18x1.45mm_HandSolder"
 			(at 81.28 66.3448 0)
 			(hide yes)
@@
 			)
 		)
-		(property "Footprint" "Resistor_SMD:R_0805_2012Metric"
+		(property "Footprint" "Capacitor_SMD:C_0805_2012Metric_Pad1.18x1.45mm_HandSolder"
 			(at 36.83 66.3448 0)
 			(hide yes)

Commit message: nvl
Parts:
- added R10, R11: 15k, Resistor_SMD:R_0805_2012Metric_Pad1.20x1.40mm_HandSolder, symbol Device:R
Connections:
- net +3.3V: now also R10.2
- net +5V: no longer C11.2, C21.1
- net GND: now also R11.1
- net at J1.1 (Pin_1), U10.3 (IN), U10.4 (IN)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: now also C11.2, C21.1
- net at A1.31 (GPIO26_ADC0): now also R10.1, R11.2; no longer U8.2 (IN2)
- net at A1.29 (GPIO22): now also U8.2 (IN2); no longer U8.3 (IN1)
- net at A1.24 (GPIO18): now also U8.3 (IN1)
Other:
- moved on the sheet: C11, C21, C7, C8, C9, J1, R7, R8, R9, U10, U13G, U13H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
