File: Schaltung (Kopie)/att.kicad_pcb (KiCad board)
At the start: 2 copper layers, 60 x 120 mm, 51 parts, among them J1 12V Power supply, J2 R&S Attenuator 26.5 GHz, J3 dB Drehgeber, J4 ESP-Controller, J5 ATT_SEL, J6 Display, U1 DRV8871DDA, U2 DRV8871DDA, U3 DRV8871DDA, U4 DRV8871DDA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

Commit message: 2
Parts:
- moved H9 169.3 mm to (152.2, 95.4)
- moved C21 100.4 mm to (34.5, 131.5), turned to -90 degrees
- moved H4 2.60 mm to (108.6, 118.0)
- moved H2 2.60 mm to (108.6, 51.7)
- moved C11 1.16 mm to (72.8, 118.0), turned to 0 degrees
- moved H3 0.90 mm to (56.7, 118.0)
Routing:
- net +5V: track 107.3 -> 165.9 mm
- net GND: track 130.8 -> 132.7 mm, vias 11 -> 13
